Commit message: pre-commit_xacro errorr

File: urdf/ur5e.urdf.xacro (robot description, xacro)
@@ -1,8 +1,9 @@
+<?xml version="1.0"?>
 <robot xmlns:xacro="http://ros.org/wiki/xacro" name="ur5e">
-  <xacro:arg name="prefix" default="ur5e_"/>
+  <!-- Include the macro and ROS 2 control definitions -->
   <xacro:include filename="$(find mujoco_accessories)/urdf/ur5e_macro.xacro"/>
   <xacro:include filename="$(find mujoco_accessories)/urdf/ur5e_ros2_control.xacro"/>
-  <!-- Apply prefix to the macro -->
-  <xacro:ur5e_macro prefix="${prefix}" />
-  <xacro:ur5e_ros2_control prefix="${prefix}" />
+  <!-- Apply the macros directly with no prefix -->
+  <xacro:ur5e_macro />
+  <xacro:ur5e_ros2_control />
 </robot>

File: urdf/ur5e_macro.xacro (robot description, xacro)
@@ -1,90 +1,118 @@
 <?xml version="1.0"?>
 <robot xmlns:xacro="http://ros.org/wiki/xacro" name="ur5e_macro">
-  <xacro:arg name="prefix" default=""/>
-  <xacro:property name="arm_length" value="1.0"/>
+  <xacro:macro name="ur5e_macro" params=""></xacro:macro>
+  <xacro:property name="arm_length" value="1.0" />
   <!-- Base Link -->
-  <link name="${prefix}base_link">
+  <link name="base_link">
     <visual>
-      <geometry><box size="0.2 0.2 0.1"/></geometry>
-      <material name="gray"><color rgba="0.5 0.5 0.5 1"/></material>
+      <geometry>
+        <box size="0.2 0.2 0.1" />
+      </geometry>
+      <material name="gray">
+        <color rgba="0.5 0.5 0.5 1" />
+      </material>
     </visual>
   </link>
   <!-- Shoulder Pan -->
-  <joint name="${prefix}shoulder_pan_joint" type="revolute">
-    <parent link="${prefix}base_link"/>
-    <child link="${prefix}shoulder_link"/>
-    <origin xyz="0 0 0.1" rpy="0 0 0"/>
-    <axis xyz="0 0 1"/>
-    <limit lower="-3.14" upper="3.14" effort="100" velocity="1.5"/>
+  <joint name="shoulder_pan_joint" type="revolute">
+    <parent link="base_link" />
+    <child link="shoulder_link" />
+    <origin xyz="0 0 0.1" rpy="0 0 0" />
+    <axis xyz="0 0 1" />
+    <limit lower="-3.14" upper="3.14" effort="100" velocity="1.5" />
   </joint>
-  <link name="${prefix}shoulder_link">
+  <link name="shoulder_link">
     <visual>
-      <geometry><cylinder length="0.2" radius="0.05"/></geometry>
-      <material name="blue"><color rgba="0.0 0.4 1.0 1"/></material>
+      <geometry>
+        <cylinder length="0.2" radius="0.05" />
+      </geometry>
+      <material name="blue">
+        <color rgba="0.0 0.4 1.0 1" />
+      </material>
     </visual>
   </link>
-  <joint name="${prefix}shoulder_lift_joint" type="revolute">
-    <parent link="${prefix}shoulder_link"/>
-    <child link="${prefix}upper_arm_link"/>
-    <origin xyz="0 0 0.2" rpy="0 0 0"/>
-    <axis xyz="0 1 0"/>
-    <limit lower="-3.14" upper="3.14" effort="100" velocity="1.5"/>
+  <joint name="shoulder_lift_joint" type="revolute">
+    <parent link="shoulder_link" />
+    <child link="upper_arm_link" />
+    <origin xyz="0 0 0.2" rpy="0 0 0" />
+    <axis xyz="0 1 0" />
+    <limit lower="-3.14" upper="3.14" effort="100" velocity="1.5" />
   </joint>
-  <link name="${prefix}upper_arm_link">
+  <link name="upper_arm_link">
     <visual>
-      <geometry><cylinder length="0.4" radius="0.04"/></geometry>
-      <material name="green"><color rgba="0.2 1.0 0.2 1"/></material>
+      <geometry>
+        <cylinder length="0.4" radius="0.04" />
+      </geometry>
+      <material name="green">
+        <color rgba="0.2 1.0 0.2 1" />
+      </material>
     </visual>
   </link>
-  <joint name="${prefix}elbow_joint" type="revolute">
-    <parent link="${prefix}upper_arm_link"/>
-    <child link="${prefix}forearm_link"/>
-    <origin xyz="0 0 0.4" rpy="0 0 0"/>
-    <axis xyz="0 1 0"/>
-    <limit lower="-3.14" upper="3.14" effort="100" velocity="1.5"/>
+  <joint name="elbow_joint" type="revolute">
+    <parent link="upper_arm_link" />
+    <child link="forearm_link" />
+    <origin xyz="0 0 0.4" rpy="0 0 0" />
+    <axis xyz="0 1 0" />
+    <limit lower="-3.14" upper="3.14" effort="100" velocity="1.5" />
   </joint>
-  <link name="${prefix}forearm_link">
+  <link name="forearm_link">
     <visual>
-      <geometry><cylinder length="0.4" radius="0.04"/></geometry>
-      <material name="red"><color rgba="1.0 0.2 0.2 1"/></material>
+      <geometry>
+        <cylinder length="0.4" radius="0.04" />
+      </geometry>
+      <material name="red">
+        <color rgba="1.0 0.2 0.2 1" />
+      </material>
     </visual>
   </link>
-  <joint name="${prefix}wrist_1_joint" type="revolute">
-    <parent link="${prefix}forearm_link"/>
-    <child link="${prefix}wrist_1_link"/>
-    <origin xyz="0 0 0.4" rpy="0 0 0"/>
-    <axis xyz="0 1 0"/>
-    <limit lower="-3.14" upper="3.14" effort="100" velocity="1.5"/>
+  <joint name="wrist_1_joint" type="revolute">
+    <parent link="forearm_link" />
+    <child link="wrist_1_link" />
+    <origin xyz="0 0 0.4" rpy="0 0 0" />
+    <axis xyz="0 1 0" />
+    <limit lower="-3.14" upper="3.14" effort="100" velocity="1.5" />
   </joint>
-  <link name="${prefix}wrist_1_link">
+  <link name="wrist_1_link">
     <visual>
-      <geometry><cylinder length="0.2" radius="0.04"/></geometry>
-      <material name="purple"><color rgba="0.5 0.0 0.5 1"/></material>
+      <geometry>
+        <cylinder length="0.2" radius="0.04" />
+      </geometry>
+      <material name="purple">
+        <color rgba="0.5 0.0 0.5 1" />
+      </material>
     </visual>
   </link>
-  <joint name="${prefix}wrist_2_joint" type="revolute">
-    <parent link="${prefix}wrist_1_link"/>
-    <child link="${prefix}wrist_2_link"/>
-    <origin xyz="0 0 0.2" rpy="0 0 0"/>
-    <axis xyz="0 1 0"/>
-    <limit lower="-3.14" upper="3.14" effort="100" velocity="1.5"/>
+  <joint name="wrist_2_joint" type="revolute">
+    <parent link="wrist_1_link" />
+    <child link="wrist_2_link" />
+    <origin xyz="0 0 0.2" rpy="0 0 0" />
+    <axis xyz="0 1 0" />
+    <limit lower="-3.14" upper="3.14" effort="100" velocity="1.5" />
   </joint>
-  <link name="${prefix}wrist_2_link">
+  <link name="wrist_2_link">
     <visual>
-      <geometry><cylinder length="0.2" radius="0.04"/></geometry>
-      <material name="yellow"><color rgba="1.0 1.0 0.0 1"/></material>
+      <geometry>
+        <cylinder length="0.2" radius="0.04" />
+      </geometry>
+      <material name="yellow">
+        <color rgba="1.0 1.0 0.0 1" />
+      </material>
     </visual>
   </link>
-  <joint name="${prefix}wrist_3_joint" type="revolute">
-    <parent link="${prefix}wrist_2_link"/>
-    <child link="${prefix}wrist_3_link"/>
-    <origin xyz="0 0 0.2" rpy="0 0 0"/>
-    <axis xyz="0 1 0"/>
-    <limit lower="-3.14" upper="3.14" effort="100" velocity="1.5"/>
+  <joint name="wrist_3_joint" type="revolute">
+    <parent link="wrist_2_link" />
+    <child link="wrist_3_link" />
+    <origin xyz="0 0 0.2" rpy="0 0 0" />
+    <axis xyz="0 1 0" />
+    <limit lower="-3.14" upper="3.14" effort="100" velocity="1.5" />
   </joint>
-  <link name="${prefix}wrist_3_link">
+  <link name="wrist_3_link">
     <visual>
-      <geometry><cylinder length="0.2" radius="0.04"/></geometry>
-      <material name="orange"><color rgba="1.0 0.5 0.0 1"/></material>
+      <geometry>
+        <cylinder length="0.2" radius="0.04" />
+      </geometry>
+      <material name="orange">
+        <color rgba="1.0 0.5 0.0 1" />
+      </material>
     </visual>
   </link>

File: urdf/ur5e_ros2_control.xacro (robot description, xacro)
@@ -1,5 +1,5 @@
 <?xml version="1.0"?>
 <robot xmlns:xacro="http://ros.org/wiki/xacro" name="ur5e_ros2_control">
-  <xacro:arg name="prefix" default=""/>
+    <xacro:macro name="ur5e_ros2_control" params=""></xacro:macro>
     <ros2_control name="ur5e" type="system">
     <hardware>
@@ -7,30 +7,30 @@
       <param name="update_rate">100</param>
     </hardware>
-    <joint name="${prefix}shoulder_pan_joint">
+    <joint name="shoulder_pan_joint">
       <command_interface name="position"/>
       <state_interface name="position"/>
       <state_interface name="velocity"/>
     </joint>
-    <joint name="${prefix}shoulder_lift_joint">
+    <joint name="shoulder_lift_joint">
       <command_interface name="position"/>
       <state_interface name="position"/>
       <state_interface name="velocity"/>
     </joint>
-    <joint name="${prefix}elbow_joint">
+    <joint name="elbow_joint">
       <command_interface name="position"/>
       <state_interface name="position"/>
       <state_interface name="velocity"/>
     </joint>
-    <joint name="${prefix}wrist_1_joint">
+    <joint name="wrist_1_joint">
       <command_interface name="position"/>
       <state_interface name="position"/>
       <state_interface name="velocity"/>
     </joint>
-    <joint name="${prefix}wrist_2_joint">
+    <joint name="wrist_2_joint">
       <command_interface name="position"/>
       <state_interface name="position"/>
       <state_interface name="velocity"/>
     </joint>
-    <joint name="${prefix}wrist_3_joint">
+    <joint name="wrist_3_joint">
       <command_interface name="position"/>
       <state_interface name="position"/>
