Commit message: final_commit_ridgeback

File: urdf/ridgeback.urdf.xacro (robot description, xacro)
@@ -1,35 +1,292 @@
 <?xml version="1.0"?>
-<robot name="ridgeback" xmlns:xacro="http://ros.org/wiki/xacro" xmlns:ros2_control="http://ros.org/schema/ros2_control">
-  <link name="base_link" />
-  <joint name="front_left_wheel" type="continuous">
+<robot name="ridgeback" xmlns:xacro="http://ros.org/wiki/xacro">
+  <xacro:property name="PI" value="3.1415926535897931" />
+  <xacro:property name="wheel_radius" value="0.0759" />
+  <xacro:property name="wheel_width" value="0.0790" />
+  <xacro:property name="chassis_length" value="0.960" />
+  <xacro:property name="chassis_width" value="0.793" />
+  <xacro:property name="chassis_height" value="0.216" />
+  <xacro:property name="deck_height" value="0.280" />
+  <xacro:property name="deck_thickness" value="0.005" />
+  <xacro:property name="riser_height" value="$(optenv RIDGEBACK_RISER_HEIGHT 0.055)" />
+  <xacro:property name="axle_offset" value="0.0500" />
+  <xacro:property name="rocker_offset" value="0.319" />
+  <xacro:property name="rocker_width" value="0.472" />
+  <xacro:property name="imu_offset_x" value="0.2085" />
+  <xacro:property name="imu_offset_y" value="-0.2902" />
+  <xacro:property name="imu_offset_z" value="0.1681" />
+  <xacro:property name="dummy_inertia" value="1e-09"/>
+  <material name="dark_grey"><color rgba="0.2 0.2 0.2 1.0" /></material>
+  <material name="light_grey"><color rgba="0.4 0.4 0.4 1.0" /></material>
+  <material name="red"><color rgba="0.8 0.0 0.0 1.0" /></material>
+  <material name="white"><color rgba="0.9 0.9 0.9 1.0" /></material>
+  <material name="yellow"><color rgba="0.8 0.8 0.0 1.0" /></material>
+  <material name="black"><color rgba="0.15 0.15 0.15 1.0" /></material>
+  <xacro:macro name="wheel" params="prefix side *joint_pose">
+    <link name="${prefix}_${side}_wheel_link">
+      <visual>
+        <origin xyz="0 0 0" rpy="${PI/2} 0 0"/>
+        <geometry>
+          <mesh filename="package://ridgeback_description/meshes/wheel.stl"/>
+        </geometry>
+        <material name="black" />
+      </visual>
+      <collision>
+        <origin xyz="0 0 0" rpy="${PI/2} 0 0"/>
+        <geometry>
+          <cylinder radius="${wheel_radius}" length="${wheel_width}"/>
+        </geometry>
+      </collision>
+      <inertial>
+        <origin xyz="0 0 0" rpy="0 0 0"/>
+        <mass value="2.3"/>
+        <inertia
+          ixx="3.3212e-3" ixy="0" ixz="0"
+          iyy="6.6424e-3" iyz="0"
+          izz="3.3212e-3"/>
+      </inertial>
+    </link>
+    <joint name="${prefix}_${side}_wheel" type="continuous">
+      <parent link="${prefix}_rocker_link"/>
+      <child link="${prefix}_${side}_wheel_link" />
+      <xacro:insert_block name="joint_pose" />
+      <axis xyz="0 1 0" />
+    </joint>
+    <transmission name="${prefix}_wheel_trans">
+      <type>transmission_interface/SimpleTransmission</type>
+      <joint name="${prefix}_${side}_wheel">
+        <hardwareInterface>hardware_interface/VelocityJointInterface</hardwareInterface>
+      </joint>
+      <actuator name="${prefix}_${side}_actuator">
+        <mechanicalReduction>1</mechanicalReduction>
+      </actuator>
+    </transmission>
+  </xacro:macro>
+  <xacro:macro name="rocker" params="prefix joint_type location *joint_limits">
+    <link name="${prefix}_rocker_link">
+      <visual>
+        <origin xyz="0 0 0" rpy="${PI/2} 0 ${PI/2}" />
+        <geometry>
+          <mesh filename="package://ridgeback_description/meshes/rocker.stl"/>
+        </geometry>
+        <material name="black" />
+      </visual>
+      <inertial>
+        <origin xyz="0 0 0" rpy="${PI/2} 0 ${PI/2}"/>
+        <mass value="10.267"/>
+        <inertia
+          ixx="0.0288" ixy="2.20484e-6" ixz="-1.3145e-5"
+          iyy="0.4324" iyz="1.8944e-3"
+          izz="0.4130"/>
+      </inertial>
+    </link>
+    <joint name="${prefix}_rocker" type="${joint_type}">
+      <parent link="axle_link"/>
+      <child link="${prefix}_rocker_link" />
+      <origin xyz="${location*rocker_offset} 0 0" rpy="0 0 0" />
+      <axis xyz="1 0 0" />
+      <xacro:insert_block name="joint_limits" />
+    </joint>
+    <xacro:wheel prefix="${prefix}" side="left">
+      <origin xyz="0 ${rocker_width/2 + wheel_width/2} 0" rpy="0 0 0" />
+    </xacro:wheel>
+    <xacro:wheel prefix="${prefix}" side="right">
+      <origin xyz="0 ${-(rocker_width/2 + wheel_width/2)} 0" rpy="0 0 0" />
+    </xacro:wheel>
+  </xacro:macro>
+  <xacro:rocker prefix="front" joint_type="revolute" location="1" >
+    <limit lower="-0.08726" upper="0.08726" effort="0" velocity="0" />
+  </xacro:rocker>
+  <xacro:rocker prefix="rear" joint_type="fixed" location="-1" >
+    <limit effort="0" velocity="0" />
+  </xacro:rocker>
+  <link name="base_link"></link>
+  <joint name="base_link_joint" type="fixed">
+    <origin xyz="0 0 0" rpy="0 0 0" />
     <parent link="base_link"/>
-    <child link="front_left_wheel_link"/>
-    <origin xyz="0 0 0" rpy="0 0 0"/>
-    <axis xyz="0 1 0"/>
-  </joint>
-  <link name="front_left_wheel_link" />
-  <joint name="front_right_wheel" type="continuous">
-    <parent link="base_link"/>
-    <child link="front_right_wheel_link"/>
-    <origin xyz="0 0 0" rpy="0 0 0"/>
-    <axis xyz="0 1 0"/>
-  </joint>
-  <link name="front_right_wheel_link" />
-  <joint name="rear_left_wheel" type="continuous">
-    <parent link="base_link"/>
-    <child link="rear_left_wheel_link"/>
-    <origin xyz="0 0 0" rpy="0 0 0"/>
-    <axis xyz="0 1 0"/>
-  </joint>
-  <link name="rear_left_wheel_link" />
-  <joint name="rear_right_wheel" type="continuous">
-    <parent link="base_link"/>
-    <child link="rear_right_wheel_link"/>
-    <origin xyz="0 0 0" rpy="0 0 0"/>
-    <axis xyz="0 1 0"/>
-  </joint>
-  <link name="rear_right_wheel_link" />
-  <ros2_control name="RidgebackHardware" type="system">
-    <hardware>
+    <child link="chassis_link" />
+  </joint>
+  <link name="chassis_link">
+    <visual>
+      <origin xyz="0 0 0" rpy="0 0 0" />
+      <geometry>
+        <mesh filename="package://ridgeback_description/meshes/body.stl"/>
+      </geometry>
+      <material name="black" />
+    </visual>
+    <collision>
+      <origin xyz="0 0 0"/>
+      <geometry>
+        <mesh filename="package://ridgeback_description/meshes/body-collision.stl"/>
+      </geometry>
+    </collision>
+    <inertial>
+      <origin xyz="0.012 0.002 0.067" rpy="${PI/2} 0 ${PI/2}"/>
+      <mass value="165.304"/>
+      <inertia
+        ixx="4.4744" ixy="0.03098" ixz="0.003647"
+        iyy="7.1624" iyz="0.1228"
+        izz="4.6155"/>
+    </inertial>
+  </link>
+  <link name="riser_link">
+    <visual>
+      <origin xyz="0 0 ${riser_height/2}" rpy="0 0 ${pi/4}" />
+      <geometry>
+        <box size="0.493 0.493 ${riser_height}" />
+      </geometry>
+      <material name="light_grey" />
+    </visual>
+    <collision>
+      <origin xyz="0 0 ${riser_height/2}" rpy="0 0 ${pi/4}" />
+      <geometry>
+        <box size="0.493 0.493 ${riser_height}" />
+      </geometry>
+    </collision>
+  </link>
+  <joint name="riser_link_joint" type="fixed">
+    <origin xyz="0 0 ${0.225 - deck_thickness}" rpy="0 0 0" />
+    <parent link="chassis_link" />
+    <child link="riser_link" />
+  </joint>
+  <joint name="right_side_cover_link_joint" type="fixed">
+    <origin xyz="0 0 0" rpy="0 0 0" />
+    <parent link="chassis_link"/>
+    <child link="right_side_cover_link" />
+  </joint>
+  <joint name="left_side_cover_link_joint" type="fixed">
+    <origin xyz="0 0 0" rpy="0 0 0" />
+    <parent link="chassis_link"/>
+    <child link="left_side_cover_link" />
+  </joint>
+  <link name="left_side_cover_link">
+    <visual>
+      <origin xyz="0 0 0" rpy="0 0 ${PI}" />
+      <geometry>
+        <mesh filename="package://ridgeback_description/meshes/side-cover.stl"/>
+      </geometry>
+      <material name="yellow" />
+    </visual>
+  </link>
+  <link name="right_side_cover_link">
+    <visual>
+      <origin xyz="0 0 0" rpy="0 0 0" />
+      <geometry>
+        <mesh filename="package://ridgeback_description/meshes/side-cover.stl"/>
+      </geometry>
+      <material name="yellow" />
+    </visual>
+  </link>
+  <joint name="front_cover_link_joint" type="fixed">
+    <origin xyz="0 0 0" rpy="0 0 0" />
+    <parent link="chassis_link"/>
+    <child link="front_cover_link" />
+  </joint>
+  <link name="front_cover_link">
+    <visual>
+      <origin xyz="0 0 0" rpy="0 0 0" />
+      <geometry>
+        <mesh filename="package://ridgeback_description/meshes/end-cover.stl" />
+      </geometry>
+      <material name="black" />
+    </visual>
+  </link>
+  <joint name="rear_cover_link_joint" type="fixed">
+    <origin xyz="0 0 0" rpy="0 0 0" />
+    <parent link="chassis_link"/>
+    <child link="rear_cover_link" />
+  </joint>
+  <link name="rear_cover_link">
+    <visual>
+      <origin xyz="0 0 0" rpy="0 0 ${PI}" />
+      <geometry>
+        <mesh filename="package://ridgeback_description/meshes/end-cover.stl" />
+      </geometry>
+      <material name="black" />
+    </visual>
+  </link>
+  <joint name="front_lights_link_joint" type="fixed">
+    <origin xyz="0 0 0" rpy="0 0 0" />
+    <parent link="chassis_link"/>
+    <child link="front_lights_link" />
+  </joint>
+  <joint name="rear_lights_link_joint" type="fixed">
+    <origin xyz="0 0 0" rpy="0 0 0" />
+    <parent link="chassis_link"/>
+    <child link="rear_lights_link" />
+  </joint>
+  <link name="front_lights_link">
+    <visual>
+      <origin xyz="0 0 0" rpy="0 0 0" />
+      <geometry>
+        <mesh filename="package://ridgeback_description/meshes/lights.stl" />
+      </geometry>
+      <material name="white" />
+    </visual>
+  </link>
+  <link name="rear_lights_link">
+    <visual>
+      <origin xyz="0 0 0" rpy="0 0 ${PI}" />
+      <geometry>
+        <mesh filename="package://ridgeback_description/meshes/lights.stl" />
+      </geometry>
+      <material name="black" />
+    </visual>
+  </link>
+  <joint name="top_link_joint" type="fixed">
+    <origin xyz="0 0 ${riser_height-deck_height+deck_thickness}" rpy="0 0 0" />
+    <parent link="riser_link"/>
+    <child link="top_link" />
+  </joint>
+  <link name="top_link">
+    <visual>
+      <origin xyz="0 0 0" rpy="0 0 0" />
+      <geometry>
+        <mesh filename="package://ridgeback_description/meshes/top.stl" />
+      </geometry>
+      <material name="black" />
+    </visual>
+    <collision>
+      <origin xyz="0 0 0" rpy="0 0 0" />
+      <geometry>
+        <mesh filename="package://ridgeback_description/meshes/top.stl"/>
+      </geometry>
+    </collision>
+  </link>
+  <joint name="axle_joint" type="fixed">
+    <origin xyz="0 0 ${axle_offset}" rpy="0 0 0" />
+    <parent link="chassis_link"/>
+    <child link="axle_link" />
+  </joint>
+  <link name="axle_link">
+    <visual>
+      <origin xyz="0 0 0" rpy="0 ${PI/2} 0" />
+      <geometry>
+        <mesh filename="package://ridgeback_description/meshes/axle.stl" />
+      </geometry>
+      <material name="black" />
+    </visual>
+  </link>
+  <link name="imu_link">
+    <inertial>
+      <mass value="0.001"/>
+      <origin xyz="0 0 0" rpy="0 0 0"/>
+      <inertia ixx="${dummy_inertia}" ixy="0.0" ixz="0.0" iyy="${dummy_inertia}" iyz="0.0" izz="${dummy_inertia}"/>
+    </inertial>
+  </link>
+  <joint name="imu_joint" type="fixed">
+    <parent link="chassis_link" />
+    <child link="imu_link" />
+    <origin xyz="${imu_offset_x} ${imu_offset_y} ${imu_offset_z}" rpy="0 0 0"/>
+  </joint>
+  <link name="mid_mount" />
+  <joint name="mid_mount_joint" type="fixed">
+    <parent link="riser_link" />
+    <child link="mid_mount" />
+    <origin xyz="0 0 ${riser_height + deck_thickness}" rpy="0 0 0"/>
+  </joint>
+  <!-- ros2_control_tags -->
+  <ros2_control name="RidgebackSystem" type="system">
+      <hardware>
       <plugin>mujoco_ros2_control/MujocoSystem</plugin>
     </hardware>
@@ -37,21 +294,25 @@
       <command_interface name="velocity"/>
       <state_interface name="position"/>
-      <state_interface name="velocity"/>
     </joint>
     <joint name="front_right_wheel">
       <command_interface name="velocity"/>
       <state_interface name="position"/>
-      <state_interface name="velocity"/>
     </joint>
     <joint name="rear_left_wheel">
       <command_interface name="velocity"/>
       <state_interface name="position"/>
-      <state_interface name="velocity"/>
     </joint>
     <joint name="rear_right_wheel">
       <command_interface name="velocity"/>
       <state_interface name="position"/>
-      <state_interface name="velocity"/>
     </joint>
   </ros2_control>
+  <!-- Bring in simulation data for Gazebo. -->
+  <!-- <xacro:include filename="$(find ridgeback_description)/urdf/ridgeback.gazebo" />
+ Optional standard accessories, including their simulation data. The rendering
+       of these into the final description is controlled by optenv variables, which
+       default each one to off.-->
+  <!-- <xacro:include filename="$(find ridgeback_description)/urdf/accessories.urdf.xacro" /> -->
+  <!-- Optional custom includes. -->
+  <!-- <xacro:include filename="$(optenv RIDGEBACK_URDF_EXTRAS empty.urdf)" /> -->
 </robot>

Commit message: combined_init

File: urdf/ridgeback.urdf.xacro (robot description, xacro)
@@ -101,8 +101,8 @@
     <limit effort="0" velocity="0" />
   </xacro:rocker>
-  <link name="base_link"></link>
+  <link name="ridgeback_base_link"></link>
   <joint name="base_link_joint" type="fixed">
     <origin xyz="0 0 0" rpy="0 0 0" />
-    <parent link="base_link"/>
+    <parent link="ridgeback_base_link"/>
     <child link="chassis_link" />
   </joint>

File: urdf/ur5e.urdf.xacro (robot description, xacro)
@@ -1,5 +1,8 @@
-<?xml version="1.0"?>
 <robot xmlns:xacro="http://ros.org/wiki/xacro" name="ur5e">
+  <xacro:arg name="prefix" default="ur5e_"/>
   <xacro:include filename="$(find mujoco_accessories)/urdf/ur5e_macro.xacro"/>
   <xacro:include filename="$(find mujoco_accessories)/urdf/ur5e_ros2_control.xacro"/>
+  <!-- Apply prefix to the macro -->
+  <xacro:ur5e_macro prefix="${prefix}" />
+  <xacro:ur5e_ros2_control prefix="${prefix}" />
 </robot>

File: urdf/ur5e_macro.xacro (robot description, xacro)
@@ -1,7 +1,8 @@
 <?xml version="1.0"?>
-<robot xmlns:xacro="http://ros.org/wiki/xacro" name="ur5e">
+<robot xmlns:xacro="http://ros.org/wiki/xacro" name="ur5e_macro">
+  <xacro:arg name="prefix" default=""/>
   <xacro:property name="arm_length" value="1.0"/>
   <!-- Base Link -->
-  <link name="base_link">
+  <link name="${prefix}base_link">
     <visual>
       <geometry><box size="0.2 0.2 0.1"/></geometry>
@@ -10,12 +11,12 @@
   </link>
   <!-- Shoulder Pan -->
-  <joint name="shoulder_pan_joint" type="revolute">
-    <parent link="base_link"/>
-    <child link="shoulder_link"/>
+  <joint name="${prefix}shoulder_pan_joint" type="revolute">
+    <parent link="${prefix}base_link"/>
+    <child link="${prefix}shoulder_link"/>
     <origin xyz="0 0 0.1" rpy="0 0 0"/>
     <axis xyz="0 0 1"/>
     <limit lower="-3.14" upper="3.14" effort="100" velocity="1.5"/>
   </joint>
-  <link name="shoulder_link">
+  <link name="${prefix}shoulder_link">
     <visual>
       <geometry><cylinder length="0.2" radius="0.05"/></geometry>
@@ -23,13 +24,12 @@
     </visual>
   </link>
-  <!-- Additional joints simplified -->
-  <joint name="shoulder_lift_joint" type="revolute">
-    <parent link="shoulder_link"/>
-    <child link="upper_arm_link"/>
+  <joint name="${prefix}shoulder_lift_joint" type="revolute">
+    <parent link="${prefix}shoulder_link"/>
+    <child link="${prefix}upper_arm_link"/>
     <origin xyz="0 0 0.2" rpy="0 0 0"/>
     <axis xyz="0 1 0"/>
     <limit lower="-3.14" upper="3.14" effort="100" velocity="1.5"/>
   </joint>
-  <link name="upper_arm_link">
+  <link name="${prefix}upper_arm_link">
     <visual>
       <geometry><cylinder length="0.4" radius="0.04"/></geometry>
@@ -37,12 +37,12 @@
     </visual>
   </link>
-  <joint name="elbow_joint" type="revolute">
-    <parent link="upper_arm_link"/>
-    <child link="forearm_link"/>
+  <joint name="${prefix}elbow_joint" type="revolute">
+    <parent link="${prefix}upper_arm_link"/>
+    <child link="${prefix}forearm_link"/>
     <origin xyz="0 0 0.4" rpy="0 0 0"/>
     <axis xyz="0 1 0"/>
     <limit lower="-3.14" upper="3.14" effort="100" velocity="1.5"/>
   </joint>
-  <link name="forearm_link">
+  <link name="${prefix}forearm_link">
     <visual>
       <geometry><cylinder length="0.4" radius="0.04"/></geometry>
@@ -50,12 +50,12 @@
     </visual>
   </link>
-  <joint name="wrist_1_joint" type="revolute">
-    <parent link="forearm_link"/>
-    <child link="wrist_1_link"/>
+  <joint name="${prefix}wrist_1_joint" type="revolute">
+    <parent link="${prefix}forearm_link"/>
+    <child link="${prefix}wrist_1_link"/>
     <origin xyz="0 0 0.4" rpy="0 0 0"/>
     <axis xyz="0 1 0"/>
     <limit lower="-3.14" upper="3.14" effort="100" velocity="1.5"/>
   </joint>
-  <link name="wrist_1_link">
+  <link name="${prefix}wrist_1_link">
     <visual>
       <geometry><cylinder length="0.2" radius="0.04"/></geometry>
@@ -63,12 +63,12 @@
     </visual>
   </link>
-  <joint name="wrist_2_joint" type="revolute">
-    <parent link="wrist_1_link"/>
-    <child link="wrist_2_link"/>
+  <joint name="${prefix}wrist_2_joint" type="revolute">
+    <parent link="${prefix}wrist_1_link"/>
+    <child link="${prefix}wrist_2_link"/>
     <origin xyz="0 0 0.2" rpy="0 0 0"/>
     <axis xyz="0 1 0"/>
     <limit lower="-3.14" upper="3.14" effort="100" velocity="1.5"/>
   </joint>
-  <link name="wrist_2_link">
+  <link name="${prefix}wrist_2_link">
     <visual>
       <geometry><cylinder length="0.2" radius="0.04"/></geometry>
@@ -76,12 +76,12 @@
     </visual>
   </link>
-  <joint name="wrist_3_joint" type="revolute">
-    <parent link="wrist_2_link"/>
-    <child link="wrist_3_link"/>
+  <joint name="${prefix}wrist_3_joint" type="revolute">
+    <parent link="${prefix}wrist_2_link"/>
+    <child link="${prefix}wrist_3_link"/>
     <origin xyz="0 0 0.2" rpy="0 0 0"/>
     <axis xyz="0 1 0"/>
     <limit lower="-3.14" upper="3.14" effort="100" velocity="1.5"/>
   </joint>
-  <link name="wrist_3_link">
+  <link name="${prefix}wrist_3_link">
     <visual>
       <geometry><cylinder length="0.2" radius="0.04"/></geometry>

File: urdf/ur5e_ros2_control.xacro (robot description, xacro)
@@ -1,35 +1,36 @@
 <?xml version="1.0"?>
 <robot xmlns:xacro="http://ros.org/wiki/xacro" name="ur5e_ros2_control">
-  <ros2_control name="ur5e" type="system">
+  <xacro:arg name="prefix" default=""/>
+    <ros2_control name="ur5e" type="system">
     <hardware>
       <plugin>mujoco_ros2_control/MujocoSystem</plugin>
       <param name="update_rate">100</param>
     </hardware>
-    <joint name="shoulder_pan_joint">
+    <joint name="${prefix}shoulder_pan_joint">
       <command_interface name="position"/>
       <state_interface name="position"/>
       <state_interface name="velocity"/>
     </joint>
-    <joint name="shoulder_lift_joint">
+    <joint name="${prefix}shoulder_lift_joint">
       <command_interface name="position"/>
       <state_interface name="position"/>
       <state_interface name="velocity"/>
     </joint>
-    <joint name="elbow_joint">
+    <joint name="${prefix}elbow_joint">
       <command_interface name="position"/>
       <state_interface name="position"/>
       <state_interface name="velocity"/>
     </joint>
-    <joint name="wrist_1_joint">
+    <joint name="${prefix}wrist_1_joint">
       <command_interface name="position"/>
       <state_interface name="position"/>
       <state_interface name="velocity"/>
     </joint>
-    <joint name="wrist_2_joint">
+    <joint name="${prefix}wrist_2_joint">
       <command_interface name="position"/>
       <state_interface name="position"/>
       <state_interface name="velocity"/>
     </joint>
-    <joint name="wrist_3_joint">
+    <joint name="${prefix}wrist_3_joint">
       <command_interface name="position"/>
       <state_interface name="position"/>

Commit message: controller_issue

File: urdf/ridgeback.urdf.xacro (robot description, xacro)
@@ -290,4 +290,5 @@
       <hardware>
       <plugin>mujoco_ros2_control/MujocoSystem</plugin>
+      <param name="resource_group">ridgeback</param>
     </hardware>
     <joint name="front_left_wheel">

File: urdf/ridgeback_ur5e.urdf.xacro (robot description, xacro)
@@ -13,5 +13,5 @@
   <joint name="ur5e_mount_joint" type="fixed">
     <parent link="mid_mount" />
-    <child link="ur5e_base_link" />
+    <child link="base_link" />
     <origin xyz="0 0 0.01" rpy="0 0 0" />
   </joint>

File: urdf/ur5e_ros2_control.xacro (robot description, xacro)
@@ -5,4 +5,5 @@
     <hardware>
       <plugin>mujoco_ros2_control/MujocoSystem</plugin>
+      <param name="resource_group">ur5e</param>
       <param name="update_rate">100</param>
     </hardware>
