Commit message: test_urdf

File: urdf/ridgeback.urdf.xacro (robot description, xacro)
@@ -28,5 +28,5 @@
         <origin xyz="0 0 0" rpy="${PI/2} 0 0"/>
         <geometry>
-          <mesh filename="package://ridgeback_description/meshes/wheel.stl"/>
+          <mesh filename="package://mujoco_accessories/meshes/ridgeback/wheel.stl"/>
         </geometry>
         <material name="black" />
@@ -68,5 +68,5 @@
         <origin xyz="0 0 0" rpy="${PI/2} 0 ${PI/2}" />
         <geometry>
-          <mesh filename="package://ridgeback_description/meshes/rocker.stl"/>
+          <mesh filename="package://mujoco_accessories/meshes/ridgeback/rocker.stl"/>
         </geometry>
         <material name="black" />
@@ -111,5 +111,5 @@
       <origin xyz="0 0 0" rpy="0 0 0" />
       <geometry>
-        <mesh filename="package://ridgeback_description/meshes/body.stl"/>
+        <mesh filename="package://mujoco_accessories/meshes/ridgeback/body.stl"/>
       </geometry>
       <material name="black" />
@@ -118,5 +118,5 @@
       <origin xyz="0 0 0"/>
       <geometry>
-        <mesh filename="package://ridgeback_description/meshes/body-collision.stl"/>
+        <mesh filename="package://mujoco_accessories/meshes/ridgeback/body-collision.stl"/>
       </geometry>
     </collision>
@@ -164,5 +164,5 @@
       <origin xyz="0 0 0" rpy="0 0 ${PI}" />
       <geometry>
-        <mesh filename="package://ridgeback_description/meshes/side-cover.stl"/>
+        <mesh filename="package://mujoco_accessories/meshes/ridgeback/side-cover.stl"/>
       </geometry>
       <material name="yellow" />
@@ -173,5 +173,5 @@
       <origin xyz="0 0 0" rpy="0 0 0" />
       <geometry>
-        <mesh filename="package://ridgeback_description/meshes/side-cover.stl"/>
+        <mesh filename="package://mujoco_accessories/meshes/ridgeback/side-cover.stl"/>
       </geometry>
       <material name="yellow" />
@@ -187,5 +187,5 @@
       <origin xyz="0 0 0" rpy="0 0 0" />
       <geometry>
-        <mesh filename="package://ridgeback_description/meshes/end-cover.stl" />
+        <mesh filename="package://mujoco_accessories/meshes/ridgeback/end-cover.stl" />
       </geometry>
       <material name="black" />
@@ -201,5 +201,5 @@
       <origin xyz="0 0 0" rpy="0 0 ${PI}" />
       <geometry>
-        <mesh filename="package://ridgeback_description/meshes/end-cover.stl" />
+        <mesh filename="package://mujoco_accessories/meshes/ridgeback/end-cover.stl" />
       </geometry>
       <material name="black" />
@@ -220,5 +220,5 @@
       <origin xyz="0 0 0" rpy="0 0 0" />
       <geometry>
-        <mesh filename="package://ridgeback_description/meshes/lights.stl" />
+        <mesh filename="package://mujoco_accessories/meshes/ridgeback/lights.stl" />
       </geometry>
       <material name="white" />
@@ -229,5 +229,5 @@
       <origin xyz="0 0 0" rpy="0 0 ${PI}" />
       <geometry>
-        <mesh filename="package://ridgeback_description/meshes/lights.stl" />
+        <mesh filename="package://mujoco_accessories/meshes/ridgeback/lights.stl" />
       </geometry>
       <material name="black" />
@@ -243,5 +243,5 @@
       <origin xyz="0 0 0" rpy="0 0 0" />
       <geometry>
-        <mesh filename="package://ridgeback_description/meshes/top.stl" />
+        <mesh filename="package://mujoco_accessories/meshes/ridgeback/top.stl" />
       </geometry>
       <material name="black" />
@@ -250,5 +250,5 @@
       <origin xyz="0 0 0" rpy="0 0 0" />
       <geometry>
-        <mesh filename="package://ridgeback_description/meshes/top.stl"/>
+        <mesh filename="package://mujoco_accessories/meshes/ridgeback/top.stl"/>
       </geometry>
     </collision>
@@ -263,5 +263,5 @@
       <origin xyz="0 0 0" rpy="0 ${PI/2} 0" />
       <geometry>
-        <mesh filename="package://ridgeback_description/meshes/axle.stl" />
+        <mesh filename="package://mujoco_accessories/meshes/ridgeback/axle.stl" />
       </geometry>
       <material name="black" />
@@ -286,5 +286,4 @@
     <origin xyz="0 0 ${riser_height + deck_thickness}" rpy="0 0 0"/>
   </joint>
-  <!-- ros2_control_tags -->
   <ros2_control name="RidgebackSystem" type="system">
       <hardware>
@@ -309,11 +308,3 @@
     </joint>
   </ros2_control>
-  <!-- Bring in simulation data for Gazebo. -->
-  <!-- <xacro:include filename="$(find ridgeback_description)/urdf/ridgeback.gazebo" />
- Optional standard accessories, including their simulation data. The rendering
-       of these into the final description is controlled by optenv variables, which
-       default each one to off.-->
-  <!-- <xacro:include filename="$(find ridgeback_description)/urdf/accessories.urdf.xacro" /> -->
-  <!-- Optional custom includes. -->
-  <!-- <xacro:include filename="$(optenv RIDGEBACK_URDF_EXTRAS empty.urdf)" /> -->
-</robot>
+  </robot>
